Commit message: Error cuando se conecta el lidar

File: kalman_description/urdf/kalman.urdf.xacro (robot description, xacro)
@@ -20,4 +20,5 @@
     </xacro:caster_wheel>
     <xacro:lidar_sensor/>
+    <xacro:imu_sensor/>
     <!--xacro:if value="$(arg use_sim)">
         <xacro:if value="$(arg use_ros2_control)">

File: kalman_description/urdf/xacro/properties.xacro (robot description, xacro)
@@ -34,3 +34,6 @@
     <xacro:property name="antena_y_offset" value="-0.031980"/>
     <xacro:property name="antena_z_offset" value="0.0706"/>
+    <xacro:property name="imu_x_offset" value="0.0"/>
+    <xacro:property name="imu_y_offset" value="0.0"/>
+    <xacro:property name="imu_z_offset" value="0.0"/>
 </robot>

File: kalman_description/urdf/xacro/sensors.xacro (robot description, xacro)
@@ -37,3 +37,36 @@
         </joint>
     </xacro:macro>
+    <xacro:macro name="imu_sensor">
+        <!--link name="laser_link">
+            <visual>
+                <origin xyz="0.0 0.0 0.0" rpy="0.0 0.0 0.0"/>
+                <geometry>
+                    <mesh filename="file://$(find kalman_description)/meshes/lidar.stl" scale="0.001 0.001 0.001"/>
+                </geometry>
+                <material name="black">
+                    <color rgba="0.0 0.0 0.0 1.0"/>
+                </material>
+            </visual>
+            <xacro:inertial_box mass="${lidar_mass}" x="${lidar_largo}" y="${lidar_ancho}" z="${lidar_altura}">
+                <origin xyz="${0.01} 0.0 ${0.0015}" rpy="0.0 0.0 0.0"/>
+            </xacro:inertial_box>
+            <collision>
+                <origin xyz="${0.01} 0.0 ${0.0015}" rpy="0.0 0.0 0.0"/>
+                <geometry>
+                    <box size="${lidar_largo} ${lidar_ancho} ${lidar_altura}"/>
+                </geometry>
+            </collision>
+        </link>
+        <joint name="base_lidar_joint" type="fixed">
+            <origin xyz="0.0 ${0.072} ${-0.1035}" rpy="0.0 0.0 ${-pi/2}"/>
+            <parent link="chassis_link"/>
+            <child link="laser_link"/>
+        </joint-->
+        <link name="imu_link"/>
+        <joint name="base_imu_joint" type="fixed">
+            <origin xyz="${imu_x_offset} ${imu_y_offset} ${imu_z_offset}" rpy="0.0 0.0 0.0"/>
+            <parent link="chassis_link"/>
+            <child link="imu_link"/>
+        </joint>
+    </xacro:macro>
 </robot>
