Commit message: feat: kalman_gazebo (con bugs por corregir para controlar el movimiento correctamente)

File: kalman_description/urdf/robot.urdf.xacro (robot description, xacro)
@@ -5,5 +5,4 @@
     <!--xacro:include filename="$(find kalman_description)/urdf/xacro/inertial.xacro"/-->
     <xacro:arg name="use_sim" default='true'  />
-    <xacro:arg name="use_ros2_control" default="true" />
     <xacro:include filename="$(find kalman_description)/urdf/xacro/chassis.xacro"/>
     <xacro:include filename="$(find kalman_description)/urdf/xacro/wheel.xacro"/>
@@ -11,5 +10,4 @@
     <xacro:include filename="$(find kalman_description)/urdf/xacro/gazebo.xacro"/>
     <xacro:include filename="$(find kalman_description)/urdf/xacro/sensors.xacro"/>
-    <xacro:include filename="$(find kalman_description)/urdf/xacro/ros2_control.xacro"/>
     <!-- Construir robot -->
     <xacro:chassis/>
@@ -21,17 +19,9 @@
     <xacro:lidar_sensor/>
     <xacro:imu_sensor/>
-    <!--xacro:if value="$(arg use_sim)">
-        <xacro:if value="$(arg use_ros2_control)">
-            <xacro:ros2_control_gazebo/>
-        </xacro:if>
-        <xacro:unless value="$(arg use_ros2_control)">
-            <xacro:gazebo_plugin_drive/>
-        </xacro:unless>
+    <xacro:if value="$(arg use_sim)">
+        <xacro:gazebo_plugin_drive/>
         <xacro:friction_gazebo/>
         <xacro:gazebo_sensors/>
         <xacro:gazebo_materials/>
-    </xacro:if-->
-    <!--xacro:unless value="$(arg use_sim)">
-        <xacro:uvrobot_ros2_control/>
-    </xacro:unless-->
+    </xacro:if>
 </robot>

File: kalman_description/urdf/xacro/gazebo.xacro (robot description, xacro)
@@ -30,78 +30,36 @@
         </gazebo>
     </xacro:macro>
-    <xacro:macro name="ros2_control_gazebo">
-        <!-- Hardware interface macro -->
-        <xacro:macro name="ros2_control" params="wheel">
-            <joint name="${wheel}_joint">
-            <command_interface name="velocity">
-                <param name="min">-10</param>
-                <param name="max">10</param>
-            </command_interface>
-            <state_interface name="position"/>
-            <state_interface name="velocity"/>
-            </joint>
-        </xacro:macro>
-        <!-- Ros2 control -->
-        <ros2_control name="GaseboSystem" type="system">
-            <hardware>
-                <plugin>gazebo_ros2_control/GazeboSystem</plugin>
-                <!--plugin>uvrobot_hardware/UVRobotHardware</plugin-->
-            </hardware>
-            <xacro:ros2_control wheel="left_wheel"/>
-            <xacro:ros2_control wheel="right_wheel"/>
-        </ros2_control>
-        <!-- Plugin ros2 control gazebo -->
-        <gazebo>
-            <plugin filename="libgazebo_ros2_control.so" name="gazebo_ros2_control">
-                <parameters>$(find uvrobot_control)/config/diff_drive_controller.yaml</parameters>
-                <ros>
-                <remapping>uvrobot_diff_base_controller/cmd_vel_unstamped:=cmd_vel</remapping>
-                <remapping>uvrobot_diff_base_controller/odom:=odom</remapping>
-                <remapping>/tf:=tf</remapping>
-                </ros>
-            </plugin>
-        </gazebo>
-    </xacro:macro>
     <xacro:macro name="gazebo_plugin_drive">
         <gazebo>
             <plugin name="differential_drive_controller" filename="libgazebo_ros_diff_drive.so">
-                <!-- Plugin update rate in Hz -->
-                <updateRate>50</updateRate>
-                <!-- Name of left joint, defaults to `left_joint` -->
-                <left_joint>left_wheel_joint</left_joint>
-                <!-- Name of right joint, defaults to `right_joint` -->
-                <right_joint>right_wheel_joint</right_joint>
-                <!-- The distance from the center of one wheel to the other, in meters, defaults to 0.34 m -->
-                <wheel_separation>0.5380</wheel_separation>
-                <!-- Diameter of the wheels, in meters, defaults to 0.15 m -->
-                <wheel_diameter>0.2410</wheel_diameter>
-                <!-- Wheel acceleration, in rad/s^2, defaults to 0.0 rad/s^2 -->
-                <wheel_acceleration>1.0</wheel_acceleration>
-                <!-- Maximum torque which the wheels can produce, in Nm, defaults to 5 Nm -->
-                <wheel_torque>20</wheel_torque>
-                <!-- Topic to receive geometry_msgs/Twist message commands, defaults to `cmd_vel` -->
+                <update_rate>30</update_rate>
+                <left_joint>wheel_left_joint</left_joint>
+                <right_joint>wheel_right_joint</right_joint>
+                <wheel_separation>${wheel_separation}</wheel_separation>
+                <wheel_diameter>${wheel_radius * 2}</wheel_diameter>
+                <max_wheel_acceleration>1.0</max_wheel_acceleration>
+                <max_wheel_torque>1.0</max_wheel_torque>
                 <command_topic>cmd_vel</command_topic>
                 <odometry_topic>odom</odometry_topic>
                 <odometry_frame>odom</odometry_frame>
-                <!-- Robot frame to calculate odometry from, defaults to `base_footprint` -->
                 <robot_base_frame>base_footprint</robot_base_frame>
-                <!-- Odometry source, 0 for ENCODER, 1 for WORLD, defaults to WORLD -->
-                <odometry_source>1</odometry_source>
-                <!-- Set to true to publish transforms for the wheel links, defaults to false -->
                 <publish_wheel_tf>true</publish_wheel_tf>
-                <!-- Set to true to publish transforms for the odometry, defaults to true -->
-                <publish_odometry_frame>true</publish_odometry_frame>
+                <publish_odom_tf>true</publish_odom_tf>
                 <publish_odom>true</publish_odom>
-                <publish_odom_tf>true</publish_odom_tf>
-                <!-- Set to true to publish sensor_msgs/JointState on /joint_states for the wheel joints, defaults to false -->
                 <publish_wheel_joint_state>true</publish_wheel_joint_state>
-                <!-- Set to true to swap right and left wheels, defaults to true -->
-                <legacy_mode>false</legacy_mode>
+                <!-- <legacy_mode>false</legacy_mode> -->
+            </plugin>
+        </gazebo>
+        <!-- Joint state publisher plugin -->
+        <gazebo>
+            <plugin name="joint_state_publisher" filename="libgazebo_ros_joint_state_publisher.so">
+                <update_rate>30</update_rate>
+                <joint_name>wheel_left_joint</joint_name>
+                <joint_name>wheel_right_joint</joint_name>
             </plugin>
         </gazebo>
     </xacro:macro>
     <xacro:macro name="friction_gazebo">
-        <!-- Friction -->
-        <gazebo reference="caster_joint">
+        <gazebo reference="caster_joint_1">
             <preserveFixedJoint>true</preserveFixedJoint>
         </gazebo>
@@ -112,40 +70,50 @@
             <mu2>0.0</mu2>
         </gazebo>
-        <gazebo reference="caster_wheel_2">
-            <kp>100000000.0</kp>
-            <kd>100000000.0</kd>
-            <mu1>0.0</mu1>
-            <mu2>0.0</mu2>
-        </gazebo>
     </xacro:macro>
     <xacro:macro name="gazebo_sensors">
         <gazebo reference="laser_link">
-            <sensor name="lidar_sensor" type="ray">
+            <sensor name="laser_scan_sensor" type="ray">
                 <always_on>1</always_on>
+                <visualize>1</visualize>
                 <update_rate>10</update_rate>
-                <visualize>0</visualize>
                 <ray>
                     <scan>
                         <horizontal>
-                            <samples>720</samples>
+                            <samples>360</samples>
                             <resolution>1</resolution>
-                            <min_angle>-${pi}</min_angle>
-                            <max_angle>${pi}</max_angle>
+                            <min_angle>0</min_angle>
+                            <max_angle>6.28319</max_angle>
                         </horizontal>
                     </scan>
                     <range>
-                        <min>0.05</min>
-                        <max>10.0</max>
-                        <resolution>0.01</resolution>
+                        <min>0.10</min>
+                        <max>12.0</max>
+                        <resolution>0.02</resolution>
                     </range>
+                    <noise>
+                        <type>gaussian</type>
+                        <mean>0</mean>
+                        <stddev>0.01</stddev>
+                    </noise>
                 </ray>
-                <plugin name="gazebo_ros_laser" filename="libgazebo_ros_ray_sensor.so">
-                    <topicName>/scan</topicName>
-                    <frameName>laser_link</frameName>
-                    <gaussianNoise>0.01</gaussianNoise>
+                <plugin name="laser_scan_plugin" filename="libgazebo_ros_ray_sensor.so">
+                    <ros>
+                        <remapping>~/out:=scan</remapping>
+                    </ros>
                     <output_type>sensor_msgs/LaserScan</output_type>
+                    <frame_name>laser_link</frame_name>
+                </plugin>
+            </sensor>
+        </gazebo>
+        <!-- IMU sensor -->
+        <gazebo reference="imu_link">
+            <sensor name="imu_sensor" type="imu">
+                <always_on>1</always_on>
+                <update_rate>50</update_rate>
+                <plugin name="imu_plugin" filename="libgazebo_ros_imu_sensor.so">
                     <ros>
-                        <remapping>/gazebo_ros_laser/out:=/scan</remapping>
+                        <remapping>~/out:=imu</remapping>
                     </ros>
+                    <frame_name>imu_link</frame_name>
                 </plugin>
             </sensor>

File: kalman_description/urdf/xacro/properties.xacro (robot description, xacro)
@@ -5,5 +5,5 @@
     <xacro:property name="chassis_y" value="0.110"/>
     <xacro:property name="chassis_z" value="0.065"/>
-    <xacro:property name="chassis_mass" value="4.0"/>
+    <xacro:property name="chassis_mass" value="1.0"/>
     <!-- Propiedades de ruedas -->
     <xacro:property name="wheel_radius" value="0.017"/>
@@ -34,4 +34,5 @@
     <xacro:property name="antena_y_offset" value="-0.031980"/>
     <xacro:property name="antena_z_offset" value="0.0706"/>
+    <!-- Propiedades del IMU -->
     <xacro:property name="imu_x_offset" value="0.0"/>
     <xacro:property name="imu_y_offset" value="0.0"/>

File: kalman_description/urdf/xacro/sensors.xacro (robot description, xacro)
@@ -5,30 +5,14 @@
     <!-- Lidar -->
     <xacro:macro name="lidar_sensor">
-        <!--link name="laser_link">
-            <visual>
+        <link name="laser_link">
+            <!-- No visual geometry - lidar is part of chassis mesh -->
+            <inertial>
                 <origin xyz="0.0 0.0 0.0" rpy="0.0 0.0 0.0"/>
-                <geometry>
-                    <mesh filename="file://$(find kalman_description)/meshes/lidar.stl" scale="0.001 0.001 0.001"/>
-                </geometry>
-                <material name="black">
-                    <color rgba="0.0 0.0 0.0 1.0"/>
-                </material>
-            </visual>
-            <xacro:inertial_box mass="${lidar_mass}" x="${lidar_largo}" y="${lidar_ancho}" z="${lidar_altura}">
-                <origin xyz="${0.01} 0.0 ${0.0015}" rpy="0.0 0.0 0.0"/>
-            </xacro:inertial_box>
-            <collision>
-                <origin xyz="${0.01} 0.0 ${0.0015}" rpy="0.0 0.0 0.0"/>
-                <geometry>
-                    <box size="${lidar_largo} ${lidar_ancho} ${lidar_altura}"/>
-                </geometry>
-            </collision>
+                <mass value="${lidar_mass}"/>
+                <inertia ixx="1e-6" ixy="0.0" ixz="0.0"
+                         iyy="1e-6" iyz="0.0"
+                         izz="1e-6"/>
+            </inertial>
         </link>
-        <joint name="base_lidar_joint" type="fixed">
-            <origin xyz="0.0 ${0.072} ${-0.1035}" rpy="0.0 0.0 ${-pi/2}"/>
-            <parent link="chassis_link"/>
-            <child link="laser_link"/>
-        </joint-->
-        <link name="laser_link"/>
         <joint name="base_lidar_joint" type="fixed">
             <origin xyz="${lidar_x_offset} ${lidar_y_offset} ${lidar_z_offset}" rpy="${pi} 0.0 -${pi/2}"/>
@@ -38,30 +22,14 @@
     </xacro:macro>
     <xacro:macro name="imu_sensor">
-        <!--link name="laser_link">
-            <visual>
+        <link name="imu_link">
+            <!-- IMU has no visual geometry - it's inside the chassis -->
+            <inertial>
                 <origin xyz="0.0 0.0 0.0" rpy="0.0 0.0 0.0"/>
-                <geometry>
-                    <mesh filename="file://$(find kalman_description)/meshes/lidar.stl" scale="0.001 0.001 0.001"/>
-                </geometry>
-                <material name="black">
-                    <color rgba="0.0 0.0 0.0 1.0"/>
-                </material>
-            </visual>
-            <xacro:inertial_box mass="${lidar_mass}" x="${lidar_largo}" y="${lidar_ancho}" z="${lidar_altura}">
-                <origin xyz="${0.01} 0.0 ${0.0015}" rpy="0.0 0.0 0.0"/>
-            </xacro:inertial_box>
-            <collision>
-                <origin xyz="${0.01} 0.0 ${0.0015}" rpy="0.0 0.0 0.0"/>
-                <geometry>
-                    <box size="${lidar_largo} ${lidar_ancho} ${lidar_altura}"/>
-                </geometry>
-            </collision>
+                <mass value="0.001"/>
+                <inertia ixx="1e-9" ixy="0.0" ixz="0.0"
+                         iyy="1e-9" iyz="0.0"
+                         izz="1e-9"/>
+            </inertial>
         </link>
-        <joint name="base_lidar_joint" type="fixed">
-            <origin xyz="0.0 ${0.072} ${-0.1035}" rpy="0.0 0.0 ${-pi/2}"/>
-            <parent link="chassis_link"/>
-            <child link="laser_link"/>
-        </joint-->
-        <link name="imu_link"/>
         <joint name="base_imu_joint" type="fixed">
             <origin xyz="${imu_x_offset} ${imu_y_offset} ${imu_z_offset}" rpy="0.0 0.0 0.0"/>

Commit message: fix: kalman_gazebo (bug: muy bajo RTF) - collisions - se agregó un caster_wheel extra

File: kalman_description/urdf/robot.urdf.xacro (robot description, xacro)
@@ -17,4 +17,7 @@
         <origin xyz="${caster_x_offset} ${caster_y_offset} ${caster_z_offset}" rpy="0 0 0"/>
     </xacro:caster_wheel>
+    <xacro:caster_wheel index="2">
+        <origin xyz="0.05 ${-caster_y_offset} ${caster_z_offset}" rpy="0 0 0"/>
+    </xacro:caster_wheel>
     <xacro:lidar_sensor/>
     <xacro:imu_sensor/>

File: kalman_description/urdf/xacro/chassis.xacro (robot description, xacro)
@@ -19,5 +19,5 @@
             </visual>
             <collision>
-                <origin xyz="0 0 0" rpy="0 0 0"/>
+                <origin xyz="0 0 -0.0155" rpy="0 0 0"/>
                 <geometry>
                     <box size="${chassis_x} ${chassis_y} ${chassis_z}"/>
@@ -49,5 +49,5 @@
                 <origin xyz="0 0 0" rpy="0 0 0"/>
                 <geometry>
-                    <cylinder radius="0.0" length="0.0"/>
+                    <cylinder radius="${antena_radius}" length="${antena_ancho}"/>
                 </geometry>
             </collision>

File: kalman_description/urdf/xacro/gazebo.xacro (robot description, xacro)
@@ -34,6 +34,8 @@
             <plugin name="differential_drive_controller" filename="libgazebo_ros_diff_drive.so">
                 <update_rate>30</update_rate>
-                <left_joint>wheel_left_joint</left_joint>
-                <right_joint>wheel_right_joint</right_joint>
+                <!-- <left_joint>wheel_left_joint</left_joint>
+                <right_joint>wheel_right_joint</right_joint> -->
+                <left_joint>wheel_right_joint</left_joint>
+                <right_joint>wheel_left_joint</right_joint>
                 <wheel_separation>${wheel_separation}</wheel_separation>
                 <wheel_diameter>${wheel_radius * 2}</wheel_diameter>
@@ -64,4 +66,8 @@
             <preserveFixedJoint>true</preserveFixedJoint>
         </gazebo>
+        <gazebo reference="caster_joint_2">
+            <preserveFixedJoint>true</preserveFixedJoint>
+        </gazebo>
+        <!-- Friction for left and right caster wheels -->
         <gazebo reference="caster_wheel_1">
             <kp>100000.0</kp>
@@ -70,4 +76,23 @@
             <mu2>0.0</mu2>
         </gazebo>
+        <gazebo reference="caster_wheel_2">
+            <kp>100000.0</kp>
+            <kd>100000.0</kd>
+            <mu1>0.0</mu1>
+            <mu2>0.0</mu2>
+        </gazebo>
+        <!-- Friction for left and right wheels -->
+        <gazebo reference="left_wheel">
+            <kp>100000.0</kp>
+            <kd>100000.0</kd>
+            <mu1>1.0</mu1>
+            <mu2>1.0</mu2>
+        </gazebo>
+        <gazebo reference="right_wheel">
+            <kp>100000.0</kp>
+            <kd>100000.0</kd>
+            <mu1>1.0</mu1>
+            <mu2>1.0</mu2>
+        </gazebo>
     </xacro:macro>
     <xacro:macro name="gazebo_sensors">
@@ -75,5 +100,5 @@
             <sensor name="laser_scan_sensor" type="ray">
                 <always_on>1</always_on>
-                <visualize>1</visualize>
+                <visualize>0</visualize>
                 <update_rate>10</update_rate>
                 <ray>

File: kalman_description/urdf/xacro/wheel.xacro (robot description, xacro)
@@ -18,5 +18,5 @@
             </visual>
             <collision>
-                <origin xyz="0 0 0" rpy="0 ${pi/2} 0"/>
+                <origin xyz="0 0 0" rpy="0 0 0"/>
                 <geometry>
                     <cylinder radius="${wheel_radius}" length="${wheel_width}"/>

Commit message: Se corrigio el description, ruedas y laser

File: kalman_description/urdf/robot.urdf.xacro (robot description, xacro)
@@ -12,6 +12,6 @@
     <!-- Construir robot -->
     <xacro:chassis/>
-    <xacro:wheel prefix="left" reflect="-1"/>
-    <xacro:wheel prefix="right" reflect="1"/>
+    <xacro:wheel prefix="left" reflect="1"/>
+    <xacro:wheel prefix="right" reflect="-1"/>
     <xacro:caster_wheel index="1">
         <origin xyz="${caster_x_offset} ${caster_y_offset} ${caster_z_offset}" rpy="0 0 0"/>

File: kalman_description/urdf/xacro/sensors.xacro (robot description, xacro)
@@ -16,5 +16,5 @@
         </link>
         <joint name="base_lidar_joint" type="fixed">
-            <origin xyz="${lidar_x_offset} ${lidar_y_offset} ${lidar_z_offset}" rpy="0.0 0.0 -${pi/2}"/>
+            <origin xyz="${lidar_x_offset} ${lidar_y_offset} ${lidar_z_offset}" rpy="-${pi} 0.0 -${pi/2}"/>
             <parent link="chassis_link"/>
             <child link="laser_link"/>
