Commit message: fix: robot_description - ya no hay warnings de color - posicion de la antena corregido

File: kalman_description/urdf/xacro/caster_wheel.xacro (robot description, xacro)
@@ -10,5 +10,7 @@
                    <mesh filename="file://$(find kalman_description)/meshes/caster_wheel.stl" scale="0.001 0.001 0.001"/>
                 </geometry>
-                <material name="black"/>
+                <material name="black">
+                    <color rgba="0.0 0.0 0.0 1.0"/>
+                </material>
             </visual>
             <collision>

File: kalman_description/urdf/xacro/properties.xacro (robot description, xacro)
@@ -31,5 +31,5 @@
     <xacro:property name="antena_radius" value="0.005" />
     <xacro:property name="antena_mass" value="0.3" />
-    <xacro:property name="antena_x_offset" value="-0.0055"/>
+    <xacro:property name="antena_x_offset" value="-0.0555"/>
     <xacro:property name="antena_y_offset" value="-0.031980"/>
     <xacro:property name="antena_z_offset" value="0.0706"/>

File: kalman_description/urdf/xacro/wheel.xacro (robot description, xacro)
@@ -13,5 +13,7 @@
                     <mesh filename="file://$(find kalman_description)/meshes/rueda.stl" scale="0.001 0.001 0.001"/>
                 </geometry>
-                <material name="black"/>
+                <material name="black">
+                    <color rgba="0.0 0.0 0.0 1.0"/>
+                </material>
             </visual>
             <collision>

Commit message: fix: kalman_gazebo ya tiene buen RTF para realizar navegación docs: readmes incompletos, ahora con contenido refactor: eliminé description de otro robot refactor: actualizacion de nombre del paquete del imu

File: kalman_description/urdf/xacro/caster_wheel.xacro (robot description, xacro)
@@ -16,6 +16,9 @@
             <collision>
                 <origin xyz="0 0 0" rpy="0 0 0"/>
+                <!-- <geometry>
+                    <mesh filename="file://$(find kalman_description)/meshes/caster_wheel.stl" scale="0.001 0.001 0.001"/>
+                </geometry> -->
                 <geometry>
-                    <mesh filename="file://$(find kalman_description)/meshes/caster_wheel.stl" scale="0.001 0.001 0.001"/>
+                    <sphere radius="${caster_radius}"/>
                 </geometry>
             </collision>
