Commit message: fix: tf del lidar feat: nueva simulación del laboratorio testeado con wall_follower

File: kalman_description/urdf/xacro/sensors.xacro (robot description, xacro)
@@ -16,5 +16,5 @@
         </link>
         <joint name="base_lidar_joint" type="fixed">
-            <origin xyz="${lidar_x_offset} ${lidar_y_offset} ${lidar_z_offset}" rpy="${pi} 0.0 -${pi/2}"/>
+            <origin xyz="${lidar_x_offset} ${lidar_y_offset} ${lidar_z_offset}" rpy="0.0 0.0 -${pi/2}"/>
             <parent link="chassis_link"/>
             <child link="laser_link"/>
